File: Eagle/passion-v2-1/passion-v2-1.sch (EAGLE design)
At the start: 108 parts, among them T1 2N7002K, T2 IRLR2905TRPBF, T3 2N7002K, T5 2N7002K, T6 2N7002K, T7 2N7002K, T9 2N7002K

Commit message: a
Parts:
- removed BAT: (no value), pinhead:PINHD-1X2
- removed C18, C19: 0.1u, rcl:C-EUC0603
- removed FT234X: (no value), pinhead:PINHD-1X4
- removed LD1117: LD1117S25_SOT223, voltage regulators:LD1117S25_SOT223
- removed LED6: (no value), led:LEDCHIPLED_0603
- removed M_L, M_R: (no value), pinhead:PINHD-2X3
- removed NJM2884: (no value), Akizuki:I-10673_NJM2884U1-33
- added BAT1: (no value), pinhead:PINHD-1X2
- added C33, C34: 0.1u, rcl:C-EUC0603
- added EC-CON-L, EC-CON-R: B4B-ZR, jst:B4B-ZR
- added JP1: (no value), pinhead:PINHD-2X3
- added LED6-1, LED6-2, LED6-3, LED6-4: (no value), led:LEDCHIPLED_0603
- added MOTOR_L, MOTOR_R: (no value), jst-ph:JST-PH2
- added NJM2884-3V3, NJM2884-5V: (no value), Akizuki:I-10673_NJM2884U1-33
- added R34, R35: 1k, rcl:R-EU_R0603
- added R38, R39, R40, R41: 470, rcl:R-EU_R0402
- added R42: 10k, rcl:R-EU_R0603
- added T4: 2N7002K, nxp_60:2N7002K
- C14: value 0.1u -> 0.33u
- C15: value 10u -> 2.2u
- C26, C27, C28, C29: value 100u -> (none)
- POWER: value EG1218S -> EG1215AA; device EG1218:EG1218S -> EG1215AA:EG1215AA
- R1: value 270 -> 10
- R11, R15: value 5.6k -> 1k
- R13, R5, R9: value 47 -> 10
- R3: value 1.5k -> 3.9k
- R33: value 0 -> 1k
- R4: value 180 -> 470
- R7: value 5.6k -> 470
Connections:
- removed net PUSH_IN_2: STM32F405RGT6.PC2/SPI2_MISO
- new net N$26: LED6-2.A, R33.2
- new net N$28: LED6-3.A, R34.2
- new net N$29: LED6-4.A, R35.2
- new net N$38: LED6-1.C, LED6-2.C, LED6-3.C, LED6-4.C, T4.D
- new net SW-POWER: POWER.2, STM32F405RGT6.PC2/SPI2_MISO
- net +3V3: now also EC-CON-L.1, EC-CON-R.1, JP1.6, NJM2884-3V3.VOUT, POWER.3, R32.1, R33.1, R34.1, R35.1, R38.2, R39.2, R40.2, R41.2; no longer NJM2884.VOUT
- net +5V: now also NJM2884-3V3.CONTROL, NJM2884-3V3.VIN, NJM2884-5V.VOUT; no longer FT234X.1, LD1117.OUT, M_L.4, M_R.4, NJM2884.CONTROL, NJM2884.VIN, R33.1, R33.2
- net +8V: now also BAT1.2, FAN.1, NJM2884-5V.CONTROL, NJM2884-5V.VIN; no longer FAN.2, LD1117.IN, POWER.O
- net EC_L_A: now also EC-CON-L.4, R41.1; no longer M_L.6
- net EC_L_B: now also EC-CON-L.3, R40.1; no longer M_L.5
- net EC_R_A: now also EC-CON-R.4, R39.1; no longer M_R.6
- net EC_R_B: now also EC-CON-R.3, R38.1; no longer M_R.5
- net GND: now also EC-CON-L.2, EC-CON-R.2, JP1.1, NJM2884-3V3.GND, NJM2884-5V.GND, T4.S; no longer FT234X.2, LD1117.GND, LED3.C, LED6.C, MODE.3, MODE.4, M_L.3, M_R.3, NJM2884.GND
- net GND2: now also BAT1.1, LED3.C, MODE.3, MODE.4, R42.1; no longer BAT.1
- net LED_6: now also T4.G; no longer R32.1
- net MOTOR_L_OUT1: now also C33.1, MOTOR_L.2; no longer C18.1, M_L.1
- net MOTOR_L_OUT2: now also C33.2, MOTOR_L.1; no longer C18.2, M_L.2
- net MOTOR_R_OUT1: now also C34.2, MOTOR_R.1; no longer C19.2, M_R.2
- net MOTOR_R_OUT2: now also C34.1, MOTOR_R.2; no longer C19.1, M_R.1
- net N$22: now also FAN.2; no longer FAN.1
- net N$30: now also POWER.1, R42.2; no longer BAT.2, POWER.P
- net N$43: now also LED6-1.A; no longer LED6.A
- net PC_RX: now also JP1.2; no longer FT234X.4
- net PC_TX: now also JP1.4; no longer FT234X.3
- net SWCL: now also JP1.3
- net SWDIO: now also JP1.5
Other:
- moved on the sheet: BOOT, C1, C10, C11, C12, C13, C14, C15, C16, C17, C2, C20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

Commit message: a
Parts:
- removed C1, C2, C3, C4: 0.1μ, rcl:C-EUC0603
- removed C26, C27, C28, C29: (no value), rcl:C-EUC1206
- removed LED_FL, LED_FR, LED_L, LED_R: (no value), led:LED5MM
- removed PT_FL, PT_FR, PT_L, PT_R: L-51ROPT1D1, lightsensor:L-51ROPT1D1
- removed R1, R13, R5, R9: 10, rcl:R-EU_R0603
- removed R10, R14, R3, R6: 3.9k, rcl:R-EU_R0603
- removed R11, R15: 1k, rcl:R-EU_R0603
- removed R12, R16, R2, R8: 10k, rcl:R-EU_R0603
- removed R4, R7: 470, rcl:R-EU_R0603
- removed T1, T3, T5, T7: 2N7002K, nxp_60:2N7002K
- added J1: B10B-ZR(LF)(SN), B10B-ZR_LF__SN_:B10B-ZR(LF)(SN)
- R19, R21, R24, R25, R26, R27, R28, R29, R30, R31, R32, R33, R34, R35: value 1k -> 470
Connections:
- removed net N$1: C26.1, LED_FL.A, R1.1
- removed net N$10: C29.1, LED_R.A, R13.1
- removed net N$11: LED_R.C, T7.D
- removed net N$12: C4.1, PT_R.E, R15.2
- removed net N$2: LED_FL.C, T1.D
- removed net N$3: C2.1, PT_FL.E, R4.2
- removed net N$4: C27.1, LED_FR.A, R5.1
- removed net N$5: LED_FR.C, T3.D
- removed net N$6: C1.1, PT_FR.E, R7.2
- removed net N$7: C28.1, LED_L.A, R9.1
- removed net N$8: LED_L.C, T5.D
- removed net N$9: C3.1, PT_L.E, R11.2
- net +3V3: now also J1.1; no longer PT_FL.C, PT_FR.C, PT_L.C, PT_R.C, R1.2, R13.2, R5.2, R9.2
- net GND: now also J1.2, LED3.C, MODE.3, MODE.4, R42.1; no longer C26.2, C27.2, C28.2, C29.2, R10.1, R11.1, R12.1, R14.1, R15.1, R16.1, R2.1, R3.1, R4.1, R6.1, R7.1, R8.1, T1.S, T3.S, T5.S, T7.S
- net GND2: no longer LED3.C, MODE.3, MODE.4, R42.1
- net IR_FL: now also J1.9; no longer R2.2, T1.G
- net IR_FR: now also J1.7; no longer R8.2, T3.G
- net IR_L: now also J1.10; no longer R12.2, T5.G
- net IR_R: now also J1.8; no longer R16.2, T7.G
- net SENSOR_FL: now also J1.4; no longer C2.2, R3.2
- net SENSOR_FR: now also J1.6; no longer C1.2, R6.2
- net SENSOR_L: now also J1.3; no longer C3.2, R10.2
- net SENSOR_R: now also J1.5; no longer C4.2, R14.2
